Commit message: Initial Commit: Added changes to integrate UR10 arm with tiger

File: robots/tiger/tiger_files/tiger_description/urdf/_ur10_tiger.xacro (robot description, xacro)
@@ -5,4 +5,8 @@
 	<xacro:include filename="$(find tiger_description)/urdf/materials.gazebo" />
 	<xacro:include filename="$(find tiger_description)/urdf/tiger_prefix.gazebo" />
+	<xacro:arg name="transmission_hw_interface" default="hardware_interface/PositionJointInterface"/>
+	<xacro:include filename="$(find ur_description)/urdf/common.gazebo.xacro" />
+	<xacro:include filename="$(find ur_description)/urdf/ur10.urdf.xacro"/>
+	<xacro:ur10_robot prefix="ur10_custom_" joint_limited="false" transmission_hw_interface="$(arg transmission_hw_interface)"/>
   <link name="world"/>
   <joint name="floating" type="floating">
@@ -10,4 +14,10 @@
 	  <child link ="base_link"/>
   </joint>
+	<!-- base link to ur10 joint-->
+	<joint name="base_link_ur10_arm_link_joint" type="fixed">
+		<parent link="base_link" />
+		<child link = "ur10_custom_base_link" />
+		<origin xyz="0.0 0.63 0.1" rpy="-${pi/2} 0.0  0.0" />
+	</joint>
 <!-- Base Link -->
   <link name="base_link">
