Commit message: changed imu parent from pelvis to r_foot

File: robots/poppy/poppy_files/poppy_description/urdf/poppy.xacro (robot description, xacro)
@@ -5,9 +5,10 @@
 	<xacro:include filename="$(find poppy_description)/urdf/materials.gazebo" />
 	<xacro:include filename="$(find poppy_description)/urdf/poppy_prefix.gazebo" />
+	<!--
 	<link name="world"/>
 	<joint name="floating" type="floating">
 		<parent link ="world"/>
 		<child link ="pelvis"/>
-	</joint>
+	</joint>-->
 	<link name="pelvis">
 		<inertial>
@@ -1035,5 +1036,5 @@
 </transmission>
 <!--sensors-->
-<xacro:imu_sensor xyz="0 0.35 0" rpy="${M_PI/2} 0 0" parent="pelvis" />
+<xacro:imu_sensor xyz="0 0.35 0" rpy="${M_PI/2} 0 0" parent="r_foot" />
 	<!-- Gazebo plugin for ROS Control -->
 	<!--
